File: KiCad/Motor.sch (KiCad schematic (older format))
At the start: 5 parts

Commit message: Added tasklist explenation
Parts:
- M1, M2: renamed from M?; footprint (none) -> Pin_Headers:Pin_Header_Angled_1x02
- R37, R38: renamed from R?; footprint (none) -> Resistors_ThroughHole:Resistor_Horizontal_RM20mm
- U6: renamed from U?; footprint (none) -> Housings_DIP:DIP-16_W7.62mm
Changed lines of the file:
@@
 $EndDescr
 $Comp
-L SN754410NE U?
+L SN754410NE U6
 U 1 1 571C28D3
 P 4850 2900
-F 0 "U?" H 5000 3500 50  0000 C CNN
+F 0 "U6" H 5000 3500 50  0000 C CNN
 F 1 "SN754410NE" H 4850 2300 50  0000 C CNN
-F 2 "" H 4850 2900 50  0000 C CNN
+F 2 "Housings_DIP:DIP-16_W7.62mm" H 4850 2900 50  0001 C CNN
 F 3 "" H 4850 2900 50  0000 C CNN
 	1    4850 2900
@@
 $EndComp
 $Comp
-L Motor M?
+L Motor M1
 U 1 1 571C29B6
 P 2650 2950
-F 0 "M?" H 2650 2850 60  0000 C CNN
+F 0 "M1" H 2650 2850 60  0000 C CNN
 F 1 "Motor" H 2650 3050 60  0000 C CNN
-F 2 "" H 2650 2950 60  0000 C CNN
+F 2 "Pin_Headers:Pin_Header_Angled_1x02" H 2650 2950 60  0001 C CNN
 F 3 "" H 2650 2950 60  0000 C CNN
 	1    2650 2950
@@
 9V
 $Comp
-L GND #PWR?
+L GND #PWR026
 U 1 1 571C303C
 P 4050 2900
-F 0 "#PWR?" H 4050 2650 50  0001 C CNN
+F 0 "#PWR026" H 4050 2650 50  0001 C CNN
 F 1 "GND" H 4050 2750 50  0000 C CNN
 F 2 "" H 4050 2900 50  0000 C CNN
@@
 $EndComp
 $Comp
-L GND #PWR?
+L GND #PWR027
 U 1 1 571C3054
 P 5650 2900
-F 0 "#PWR?" H 5650 2650 50  0001 C CNN
+F 0 "#PWR027" H 5650 2650 50  0001 C CNN
 F 1 "GND" H 5650 2750 50  0000 C CNN
 F 2 "" H 5650 2900 50  0000 C CNN
@@
 5V
 $Comp
-L Motor M?
+L Motor M2
 U 1 1 571C3169
 P 7050 2950
-F 0 "M?" H 7050 2850 60  0000 C CNN
+F 0 "M2" H 7050 2850 60  0000 C CNN
 F 1 "Motor" H 7050 3050 60  0000 C CNN
-F 2 "" H 7050 2950 60  0000 C CNN
+F 2 "Pin_Headers:Pin_Header_Angled_1x02" H 7050 2950 60  0001 C CNN
 F 3 "" H 7050 2950 60  0000 C CNN
 	1    7050 2950
@@
 	6400 2400 7050 2400
 $Comp
-L R R?
+L R R37
 U 1 1 571DE5C4
 P 6050 2700
-F 0 "R?" V 6130 2700 50  0000 C CNN
+F 0 "R37" V 6130 2700 50  0000 C CNN
 F 1 "56" V 6050 2700 50  0000 C CNN
-F 2 "" V 5980 2700 50  0000 C CNN
+F 2 "Resistors_ThroughHole:Resistor_Horizontal_RM20mm" V 5980 2700 50  0001 C CNN
 F 3 "" H 6050 2700 50  0000 C CNN
 	1    6050 2700
@@
 $EndComp
 $Comp
-L R R?
+L R R38
 U 1 1 571DE5F1
 P 6050 3100
-F 0 "R?" V 6130 3100 50  0000 C CNN
+F 0 "R38" V 6130 3100 50  0000 C CNN
 F 1 "56" V 6050 3100 50  0000 C CNN
-F 2 "" V 5980 3100 50  0000 C CNN
+F 2 "Resistors_ThroughHole:Resistor_Horizontal_RM20mm" V 5980 3100 50  0001 C CNN
 F 3 "" H 6050 3100 50  0000 C CNN
 	1    6050 3100
