File: KiCad/Motor.sch (KiCad schematic (older format))
At the start: 3 parts

Commit message: CHange in motorSchematics
Parts:
- added R? (x2): 47, symbol R
Connections:
- net at U?.11 (3Y): now also R?.2; no longer M?.1
- net at U?.14 (4Y): now also R?.2; no longer M?.2
- new net: M?.1, R?.1
- new net: M?.2, R?.1
Changed lines of the file:
@@
 	6400 2400 6400 2700
-Wire Wire Line
-	6400 2700 5550 2700
 Wire Wire Line
 	7050 3500 6400 3500
 Wire Wire Line
 	6400 3500 6400 3100
+$Comp
+L R R?
+U 1 1 571CA76A
+P 6000 3100
+F 0 "R?" V 6080 3100 50  0000 C CNN
+F 1 "47" V 6000 3100 50  0000 C CNN
+F 2 "" V 5930 3100 50  0000 C CNN
+F 3 "" H 6000 3100 50  0000 C CNN
+	1    6000 3100
+	0    1    1    0
+$EndComp
 Wire Wire Line
-	6400 3100 5550 3100
+	5850 3100 5550 3100
+Wire Wire Line
+	6400 3100 6150 3100
+$Comp
+L R R?
+U 1 1 571CA7D8
+P 6000 2700
+F 0 "R?" V 6080 2700 50  0000 C CNN
+F 1 "47" V 6000 2700 50  0000 C CNN
+F 2 "" V 5930 2700 50  0000 C CNN
+F 3 "" H 6000 2700 50  0000 C CNN
+	1    6000 2700
+	0    1    1    0
+$EndComp
+Wire Wire Line
+	5850 2700 5550 2700
+Wire Wire Line
+	6400 2700 6150 2700
 $EndSCHEMATC

Commit message: Changed values of resistors
Parts:
- removed R? (x2): 47, symbol R
- added R? (x2): 56, symbol R
Connections:
- net at U?.11 (3Y): now also R?.2
- net at U?.14 (4Y): now also R?.2
- net Vroom: now reaches M?.2, U?.3 (1Y)
- net at M?.1: now also R?.1
- net Styrning: now reaches M?.2
- net Styrning: now also R?.1
Changed lines of the file:
@@
 Text HLabel 4150 3400 0    60   Input ~ 0
 9V
-Wire Wire Line
-	2650 2400 3300 2400
-Wire Wire Line
-	3300 2400 3300 2700
-Wire Wire Line
-	3300 2700 4150 2700
-Wire Wire Line
-	2650 3500 3300 3500
-Wire Wire Line
-	3300 3500 3300 3100
-Wire Wire Line
-	3300 3100 4150 3100
-Wire Wire Line
-	5650 2400 5550 2400
-Wire Wire Line
-	4150 2100 4150 2400
-Connection ~ 5600 2400
-Wire Wire Line
-	5600 2400 5600 2100
-Wire Wire Line
-	5600 2100 4150 2100
 $Comp
 L GND #PWR?
@@
 	0    -1   -1   0
 $EndComp
-Wire Wire Line
-	5650 2850 5650 2950
-Wire Wire Line
-	5650 2850 5550 2850
-Wire Wire Line
-	5650 2950 5550 2950
-Connection ~ 5650 2900
-Wire Wire Line
-	4150 2850 4050 2850
-Wire Wire Line
-	4050 2850 4050 2950
-Wire Wire Line
-	4050 2950 4150 2950
-Connection ~ 4050 2900
 Text HLabel 5550 2550 2    60   Input ~ 0
 Right
@@
 $EndComp
 Wire Wire Line
+	2650 2400 3300 2400
+Wire Wire Line
+	3300 2400 3300 2700
+Wire Wire Line
+	3300 2700 4150 2700
+Wire Wire Line
+	2650 3500 3300 3500
+Wire Wire Line
+	3300 3500 3300 3100
+Wire Wire Line
+	3300 3100 4150 3100
+Wire Wire Line
+	5650 2400 5550 2400
+Wire Wire Line
+	4150 2100 4150 2400
+Connection ~ 5600 2400
+Wire Wire Line
+	5600 2400 5600 2100
+Wire Wire Line
+	5600 2100 4150 2100
+Wire Wire Line
+	5650 2850 5650 2950
+Wire Wire Line
+	5650 2850 5550 2850
+Wire Wire Line
+	5650 2950 5550 2950
+Connection ~ 5650 2900
+Wire Wire Line
+	4150 2850 4050 2850
+Wire Wire Line
+	4050 2850 4050 2950
+Wire Wire Line
+	4050 2950 4150 2950
+Connection ~ 4050 2900
+Wire Wire Line
+	6400 3100 6400 3500
+Wire Wire Line
+	6400 3500 7050 3500
+Wire Wire Line
+	6400 2700 6400 2400
+Wire Wire Line
 	6400 2400 7050 2400
-Wire Wire Line
-	6400 2400 6400 2700
-Wire Wire Line
-	7050 3500 6400 3500
-Wire Wire Line
-	6400 3500 6400 3100
 $Comp
 L R R?
-U 1 1 571CA76A
-P 6000 3100
-F 0 "R?" V 6080 3100 50  0000 C CNN
-F 1 "47" V 6000 3100 50  0000 C CNN
-F 2 "" V 5930 3100 50  0000 C CNN
-F 3 "" H 6000 3100 50  0000 C CNN
-	1    6000 3100
+U 1 1 571DE5C4
+P 6050 2700
+F 0 "R?" V 6130 2700 50  0000 C CNN
+F 1 "56" V 6050 2700 50  0000 C CNN
+F 2 "" V 5980 2700 50  0000 C CNN
+F 3 "" H 6050 2700 50  0000 C CNN
+	1    6050 2700
+	0    1    1    0
+$EndComp
+$Comp
+L R R?
+U 1 1 571DE5F1
+P 6050 3100
+F 0 "R?" V 6130 3100 50  0000 C CNN
+F 1 "56" V 6050 3100 50  0000 C CNN
+F 2 "" V 5980 3100 50  0000 C CNN
+F 3 "" H 6050 3100 50  0000 C CNN
+	1    6050 3100
 	0    1    1    0
 $EndComp
 Wire Wire Line
-	5850 3100 5550 3100
+	6400 3100 6200 3100
 Wire Wire Line
-	6400 3100 6150 3100
-$Comp
-L R R?
-U 1 1 571CA7D8
-P 6000 2700
-F 0 "R?" V 6080 2700 50  0000 C CNN
-F 1 "47" V 6000 2700 50  0000 C CNN
-F 2 "" V 5930 2700 50  0000 C CNN
-F 3 "" H 6000 2700 50  0000 C CNN
-	1    6000 2700
-	0    1    1    0
-$EndComp
+	6400 2700 6200 2700
 Wire Wire Line
-	5850 2700 5550 2700
+	5900 2700 5550 2700
 Wire Wire Line
-	6400 2700 6150 2700
+	5900 3100 5550 3100
+Text Label 2800 2400 0    60   ~ 0
+Vroom
+Text Label 6550 2400 0    60   ~ 0
+Styrning
 $EndSCHEMATC

Commit message: Updated the schematics and started with the PCB
Parts:
- R38, R39: renamed from R?; footprint (none) -> Resistors_ThroughHole:Resistor_Vertical_RM5mm
- U6: renamed from U?; footprint (none) -> Housings_DIP:DIP-16_W7.62mm_LongPads
- gave numbers to parts that had none: 2
Connections:
- net labels removed: GND
Changed lines of the file:
@@
 $Descr A4 11693 8268
 encoding utf-8
-Sheet 7 7
+Sheet 7 6
 Title ""
 Date ""
@@
 $EndDescr
 $Comp
-L SN754410NE U?
+L SN754410NE U6
 U 1 1 571C28D3
 P 4850 2900
-F 0 "U?" H 5000 3500 50  0000 C CNN
+F 0 "U6" H 5000 3500 50  0000 C CNN
 F 1 "SN754410NE" H 4850 2300 50  0000 C CNN
-F 2 "" H 4850 2900 50  0000 C CNN
+F 2 "Housings_DIP:DIP-16_W7.62mm_LongPads" H 4850 2900 50  0001 C CNN
 F 3 "" H 4850 2900 50  0000 C CNN
 	1    4850 2900
@@
 $EndComp
 $Comp
-L Motor M?
+L Motor M1
 U 1 1 571C29B6
 P 2650 2950
-F 0 "M?" H 2650 2850 60  0000 C CNN
+F 0 "M1" H 2650 2850 60  0000 C CNN
 F 1 "Motor" H 2650 3050 60  0000 C CNN
-F 2 "" H 2650 2950 60  0000 C CNN
 F 3 "" H 2650 2950 60  0000 C CNN
 	1    2650 2950
@@
 9V
 $Comp
-L GND #PWR?
 U 1 1 571C303C
 P 4050 2900
-F 0 "#PWR?" H 4050 2650 50  0001 C CNN
 F 1 "GND" H 4050 2750 50  0000 C CNN
 F 2 "" H 4050 2900 50  0000 C CNN
@@
 $EndComp
 $Comp
-L GND #PWR?
 U 1 1 571C3054
 P 5650 2900
-F 0 "#PWR?" H 5650 2650 50  0001 C CNN
 F 1 "GND" H 5650 2750 50  0000 C CNN
 F 2 "" H 5650 2900 50  0000 C CNN
@@
 5V
 $Comp
-L Motor M?
+L Motor M2
 U 1 1 571C3169
 P 7050 2950
-F 0 "M?" H 7050 2850 60  0000 C CNN
+F 0 "M2" H 7050 2850 60  0000 C CNN
 F 1 "Motor" H 7050 3050 60  0000 C CNN
-F 2 "" H 7050 2950 60  0000 C CNN
 F 3 "" H 7050 2950 60  0000 C CNN
 	1    7050 2950
@@
 	6400 2400 7050 2400
 $Comp
-L R R?
+L R R38
 U 1 1 571DE5C4
 P 6050 2700
-F 0 "R?" V 6130 2700 50  0000 C CNN
+F 0 "R38" V 6130 2700 50  0000 C CNN
 F 1 "56" V 6050 2700 50  0000 C CNN
-F 2 "" V 5980 2700 50  0000 C CNN
+F 2 "Resistors_ThroughHole:Resistor_Vertical_RM5mm" V 5980 2700 50  0001 C CNN
 F 3 "" H 6050 2700 50  0000 C CNN
 	1    6050 2700
@@
 $EndComp
 $Comp
-L R R?
+L R R39
 U 1 1 571DE5F1
 P 6050 3100
-F 0 "R?" V 6130 3100 50  0000 C CNN
+F 0 "R39" V 6130 3100 50  0000 C CNN
 F 1 "56" V 6050 3100 50  0000 C CNN
-F 2 "" V 5980 3100 50  0000 C CNN
+F 2 "Resistors_ThroughHole:Resistor_Vertical_RM5mm" V 5980 3100 50  0001 C CNN
 F 3 "" H 6050 3100 50  0000 C CNN
 	1    6050 3100

Commit message: Added two files to comit
Parts:
- M1, M2: footprint (none) -> Wire_Connections_Bridges:WireConnection_1.50mmDrill
Connections:
- net labels added: GND
Changed lines of the file:
@@
 F 0 "M1" H 2650 2850 60  0000 C CNN
 F 1 "Motor" H 2650 3050 60  0000 C CNN
+F 2 "Wire_Connections_Bridges:WireConnection_1.50mmDrill" H 2650 2950 60  0001 C CNN
 F 3 "" H 2650 2950 60  0000 C CNN
 	1    2650 2950
@@
 9V
 $Comp
+L GND #PWR026
 U 1 1 571C303C
 P 4050 2900
+F 0 "#PWR026" H 4050 2650 50  0001 C CNN
 F 1 "GND" H 4050 2750 50  0000 C CNN
 F 2 "" H 4050 2900 50  0000 C CNN
@@
 $EndComp
 $Comp
+L GND #PWR027
 U 1 1 571C3054
 P 5650 2900
+F 0 "#PWR027" H 5650 2650 50  0001 C CNN
 F 1 "GND" H 5650 2750 50  0000 C CNN
 F 2 "" H 5650 2900 50  0000 C CNN
@@
 F 0 "M2" H 7050 2850 60  0000 C CNN
 F 1 "Motor" H 7050 3050 60  0000 C CNN
+F 2 "Wire_Connections_Bridges:WireConnection_1.50mmDrill" H 7050 2950 60  0001 C CNN
 F 3 "" H 7050 2950 60  0000 C CNN
 	1    7050 2950

Commit message: Added smaller footprints
Parts:
- M1, M2: footprint Wire_Connections_Bridges:WireConnection_1.50mmDrill -> Wire_Pads:SolderWirePad_2x_1mmDrill
Changed lines of the file:
@@
 F 0 "M1" H 2650 2850 60  0000 C CNN
 F 1 "Motor" H 2650 3050 60  0000 C CNN
-F 2 "Wire_Connections_Bridges:WireConnection_1.50mmDrill" H 2650 2950 60  0001 C CNN
+F 2 "Wire_Pads:SolderWirePad_2x_1mmDrill" H 2650 2950 60  0001 C CNN
 F 3 "" H 2650 2950 60  0000 C CNN
 	1    2650 2950
@@
 9V
 $Comp
-L GND #PWR22
+L GND #PWR022
 U 1 1 571C303C
 P 4050 2900
-F 0 "#PWR22" H 4050 2650 50  0001 C CNN
+F 0 "#PWR022" H 4050 2650 50  0001 C CNN
 F 1 "GND" H 4050 2750 50  0000 C CNN
 F 2 "" H 4050 2900 50  0000 C CNN
@@
 $EndComp
 $Comp
-L GND #PWR23
+L GND #PWR023
 U 1 1 571C3054
 P 5650 2900
-F 0 "#PWR23" H 5650 2650 50  0001 C CNN
+F 0 "#PWR023" H 5650 2650 50  0001 C CNN
 F 1 "GND" H 5650 2750 50  0000 C CNN
 F 2 "" H 5650 2900 50  0000 C CNN
@@
 F 0 "M2" H 7050 2850 60  0000 C CNN
 F 1 "Motor" H 7050 3050 60  0000 C CNN
-F 2 "Wire_Connections_Bridges:WireConnection_1.50mmDrill" H 7050 2950 60  0001 C CNN
+F 2 "Wire_Pads:SolderWirePad_2x_1mmDrill" H 7050 2950 60  0001 C CNN
 F 3 "" H 7050 2950 60  0000 C CNN
 	1    7050 2950

Commit message: Revert "Added smaller footprints"
This reverts commit 0613a684753a289cb87120d105616d3a60c555f9.
Parts:
- M1, M2: footprint Wire_Pads:SolderWirePad_2x_1mmDrill -> Wire_Connections_Bridges:WireConnection_1.50mmDrill
Changed lines of the file:
@@
 F 0 "M1" H 2650 2850 60  0000 C CNN
 F 1 "Motor" H 2650 3050 60  0000 C CNN
-F 2 "Wire_Pads:SolderWirePad_2x_1mmDrill" H 2650 2950 60  0001 C CNN
+F 2 "Wire_Connections_Bridges:WireConnection_1.50mmDrill" H 2650 2950 60  0001 C CNN
 F 3 "" H 2650 2950 60  0000 C CNN
 	1    2650 2950
@@
 9V
 $Comp
-L GND #PWR022
+L GND #PWR22
 U 1 1 571C303C
 P 4050 2900
-F 0 "#PWR022" H 4050 2650 50  0001 C CNN
+F 0 "#PWR22" H 4050 2650 50  0001 C CNN
 F 1 "GND" H 4050 2750 50  0000 C CNN
 F 2 "" H 4050 2900 50  0000 C CNN
@@
 $EndComp
 $Comp
-L GND #PWR023
+L GND #PWR23
 U 1 1 571C3054
 P 5650 2900
-F 0 "#PWR023" H 5650 2650 50  0001 C CNN
+F 0 "#PWR23" H 5650 2650 50  0001 C CNN
 F 1 "GND" H 5650 2750 50  0000 C CNN
 F 2 "" H 5650 2900 50  0000 C CNN
@@
 F 0 "M2" H 7050 2850 60  0000 C CNN
 F 1 "Motor" H 7050 3050 60  0000 C CNN
-F 2 "Wire_Pads:SolderWirePad_2x_1mmDrill" H 7050 2950 60  0001 C CNN
+F 2 "Wire_Connections_Bridges:WireConnection_1.50mmDrill" H 7050 2950 60  0001 C CNN
 F 3 "" H 7050 2950 60  0000 C CNN
 	1    7050 2950
