File: KiCad/Motor.sch (KiCad schematic (older format))
At the start: 5 parts, among them M1 Motor, M2 Motor, U6 SN754410NE

Commit message: Updated the pcb to smaller size and footprints
Parts:
- M1, M2: footprint Wire_Pads:SolderWirePad_2x_1mmDrill -> Holes:SolderWirePad1mmmodified
Changed lines of the file:
@@
 F 0 "M1" H 2650 2850 60  0000 C CNN
 F 1 "Motor" H 2650 3050 60  0000 C CNN
-F 2 "Wire_Pads:SolderWirePad_2x_1mmDrill" H 2650 2950 60  0001 C CNN
+F 2 "Holes:SolderWirePad1mmmodified" H 2650 2950 60  0001 C CNN
 F 3 "" H 2650 2950 60  0000 C CNN
 	1    2650 2950
@@
 Text HLabel 4150 3250 0    60   Input ~ 0
 Backw.
-Text HLabel 5650 2400 2    60   Input ~ 0
+Text HLabel 5550 2400 2    60   Input ~ 0
 5V
 Text HLabel 4150 3400 0    60   Input ~ 0
 9V
 $Comp
-L GND #PWR022
+L GND #PWR024
 U 1 1 571C303C
-P 4050 2900
-F 0 "#PWR022" H 4050 2650 50  0001 C CNN
-F 1 "GND" H 4050 2750 50  0000 C CNN
-F 2 "" H 4050 2900 50  0000 C CNN
-F 3 "" H 4050 2900 50  0000 C CNN
-	1    4050 2900
+P 4150 2850
+F 0 "#PWR024" H 4150 2600 50  0001 C CNN
+F 1 "GND" H 4150 2700 50  0000 C CNN
+F 2 "" H 4150 2850 50  0000 C CNN
+F 3 "" H 4150 2850 50  0000 C CNN
+	1    4150 2850
 	0    1    1    0
 $EndComp
 $Comp
-L GND #PWR023
+L GND #PWR025
 U 1 1 571C3054
-P 5650 2900
-F 0 "#PWR023" H 5650 2650 50  0001 C CNN
-F 1 "GND" H 5650 2750 50  0000 C CNN
-F 2 "" H 5650 2900 50  0000 C CNN
-F 3 "" H 5650 2900 50  0000 C CNN
-	1    5650 2900
+P 5550 2950
+F 0 "#PWR025" H 5550 2700 50  0001 C CNN
+F 1 "GND" H 5550 2800 50  0000 C CNN
+F 2 "" H 5550 2950 50  0000 C CNN
+F 3 "" H 5550 2950 50  0000 C CNN
+	1    5550 2950
 	0    -1   -1   0
 $EndComp
@@
 F 0 "M2" H 7050 2850 60  0000 C CNN
 F 1 "Motor" H 7050 3050 60  0000 C CNN
-F 2 "Wire_Pads:SolderWirePad_2x_1mmDrill" H 7050 2950 60  0001 C CNN
+F 2 "Holes:SolderWirePad1mmmodified" H 7050 2950 60  0001 C CNN
 F 3 "" H 7050 2950 60  0000 C CNN
 	1    7050 2950
@@
 Wire Wire Line
 	3300 3100 4150 3100
-Wire Wire Line
-	5650 2400 5550 2400
-Wire Wire Line
-	4150 2100 4150 2400
-Connection ~ 5600 2400
-Wire Wire Line
-	5600 2400 5600 2100
-Wire Wire Line
-	5600 2100 4150 2100
-Wire Wire Line
-	5650 2850 5650 2950
-Wire Wire Line
-	5650 2850 5550 2850
-Wire Wire Line
-	5650 2950 5550 2950
-Connection ~ 5650 2900
-Wire Wire Line
-	4150 2850 4050 2850
-Wire Wire Line
-	4050 2850 4050 2950
-Wire Wire Line
-	4050 2950 4150 2950
-Connection ~ 4050 2900
 Wire Wire Line
 	6400 3100 6400 3500
@@
 Text Label 6550 2400 0    60   ~ 0
 Styrning
+$Comp
+L GND #PWR026
+U 1 1 573E2A4D
+P 4150 2950
+F 0 "#PWR026" H 4150 2700 50  0001 C CNN
+F 1 "GND" H 4150 2800 50  0000 C CNN
+F 2 "" H 4150 2950 50  0000 C CNN
+F 3 "" H 4150 2950 50  0000 C CNN
+	1    4150 2950
+	0    1    1    0
+$EndComp
+$Comp
+L GND #PWR027
+U 1 1 573E2B1A
+P 5550 2850
+F 0 "#PWR027" H 5550 2600 50  0001 C CNN
+F 1 "GND" H 5550 2700 50  0000 C CNN
+F 2 "" H 5550 2850 50  0000 C CNN
+F 3 "" H 5550 2850 50  0000 C CNN
+	1    5550 2850
+	0    -1   -1   0
+$EndComp
+Text HLabel 4150 2400 0    60   Input ~ 0
+5V
 $EndSCHEMATC
