File: KiCad/OpAmp.sch (KiCad schematic (older format))
At the start: 7 parts

Commit message: Added tasklist explenation
Parts:
- R22, R23, R24, R25, R26, R27: renamed from R?; footprint (none) -> Resistors_ThroughHole:Resistor_Horizontal_RM20mm
- U4: renamed from U?; footprint (none) -> Housings_DIP:DIP-8_W7.62mm
Changed lines of the file:
@@
 $EndDescr
 $Comp
-L CA3240E U?
+L CA3240E U4
 U 1 1 5718642F
 P 4150 1900
-F 0 "U?" H 3850 2250 50  0000 L CNN
+F 0 "U4" H 3850 2250 50  0000 L CNN
 F 1 "CA3240E" H 3850 1550 50  0000 L CNN
-F 2 "" H 4150 1900 50  0000 C CNN
+F 2 "Housings_DIP:DIP-8_W7.62mm" H 4150 1900 50  0001 C CNN
 F 3 "" H 4150 1900 50  0000 C CNN
 	1    4150 1900
@@
 SignalIn(B)
 $Comp
-L R R?
+L R R24
 U 1 1 571877CF
 P 3250 1700
-F 0 "R?" V 3330 1700 50  0000 C CNN
+F 0 "R24" V 3330 1700 50  0000 C CNN
 F 1 "150" V 3250 1700 50  0000 C CNN
-F 2 "" V 3180 1700 50  0000 C CNN
+F 2 "Resistors_ThroughHole:Resistor_Horizontal_RM20mm" V 3180 1700 50  0001 C CNN
 F 3 "" H 3250 1700 50  0000 C CNN
 	1    3250 1700
@@
 $EndComp
 $Comp
-L R R?
+L R R23
 U 1 1 57187832
 P 3000 2400
-F 0 "R?" V 3080 2400 50  0000 C CNN
+F 0 "R23" V 3080 2400 50  0000 C CNN
 F 1 "100" V 3000 2400 50  0000 C CNN
-F 2 "" V 2930 2400 50  0000 C CNN
+F 2 "Resistors_ThroughHole:Resistor_Horizontal_RM20mm" V 2930 2400 50  0001 C CNN
 F 3 "" H 3000 2400 50  0000 C CNN
 	1    3000 2400
@@
 $EndComp
 $Comp
-L GND #PWR?
+L GND #PWR017
 U 1 1 571879D5
 P 3000 2550
-F 0 "#PWR?" H 3000 2300 50  0001 C CNN
+F 0 "#PWR017" H 3000 2300 50  0001 C CNN
 F 1 "GND" H 3000 2400 50  0000 C CNN
 F 2 "" H 3000 2550 50  0000 C CNN
@@
 $EndComp
 $Comp
-L GND #PWR?
+L GND #PWR018
 U 1 1 571879F0
 P 3700 2200
-F 0 "#PWR?" H 3700 1950 50  0001 C CNN
+F 0 "#PWR018" H 3700 1950 50  0001 C CNN
 F 1 "GND" H 3700 2050 50  0000 C CNN
 F 2 "" H 3700 2200 50  0000 C CNN
@@
 	4550 1850 4950 1850
 $Comp
-L R R?
+L R R25
 U 1 1 57187D93
 P 5100 1850
-F 0 "R?" V 5180 1850 50  0000 C CNN
+F 0 "R25" V 5180 1850 50  0000 C CNN
 F 1 "150" V 5100 1850 50  0000 C CNN
-F 2 "" V 5030 1850 50  0000 C CNN
+F 2 "Resistors_ThroughHole:Resistor_Horizontal_RM20mm" V 5030 1850 50  0001 C CNN
 F 3 "" H 5100 1850 50  0000 C CNN
 	1    5100 1850
@@
 Connection ~ 4850 1850
 $Comp
-L GND #PWR?
+L GND #PWR019
 U 1 1 57187F37
 P 5400 2550
-F 0 "#PWR?" H 5400 2300 50  0001 C CNN
+F 0 "#PWR019" H 5400 2300 50  0001 C CNN
 F 1 "GND" H 5400 2400 50  0000 C CNN
 F 2 "" H 5400 2550 50  0000 C CNN
@@
 	4850 1950 4850 2200
 $Comp
-L R R?
+L R R27
 U 1 1 571881CA
 P 5400 2400
-F 0 "R?" V 5480 2400 50  0000 C CNN
+F 0 "R27" V 5480 2400 50  0000 C CNN
 F 1 "100" V 5400 2400 50  0000 C CNN
-F 2 "" V 5330 2400 50  0000 C CNN
+F 2 "Resistors_ThroughHole:Resistor_Horizontal_RM20mm" V 5330 2400 50  0001 C CNN
 F 3 "" H 5400 2400 50  0000 C CNN
 	1    5400 2400
@@
 $EndComp
 $Comp
-L R R?
+L R R26
 U 1 1 57188573
 P 5400 2000
-F 0 "R?" V 5480 2000 50  0000 C CNN
+F 0 "R26" V 5480 2000 50  0000 C CNN
 F 1 "150" V 5400 2000 50  0000 C CNN
-F 2 "" V 5330 2000 50  0000 C CNN
+F 2 "Resistors_ThroughHole:Resistor_Horizontal_RM20mm" V 5330 2000 50  0001 C CNN
 F 3 "" H 5400 2000 50  0000 C CNN
 	1    5400 2000
@@
 Connection ~ 5400 2200
 $Comp
-L R R?
+L R R22
 U 1 1 57188968
 P 3000 1850
-F 0 "R?" V 3080 1850 50  0000 C CNN
+F 0 "R22" V 3080 1850 50  0000 C CNN
 F 1 "150" V 3000 1850 50  0000 C CNN
-F 2 "" V 2930 1850 50  0000 C CNN
+F 2 "Resistors_ThroughHole:Resistor_Horizontal_RM20mm" V 2930 1850 50  0001 C CNN
 F 3 "" H 3000 1850 50  0000 C CNN
 	1    3000 1850
