File: KiCad/Project.sch (KiCad schematic (older format))
At the start: 6 parts, among them IC1 ATMEGA328-P, U1 BlueSmirf

Commit message: Added tasklist explenation
Parts:
- IC1: footprint DIL28 -> Housings_DIP:DIP-28_W7.62mm
- Q1: renamed from Q?; footprint (none) -> TO_SOT_Packages_THT:TO-92_Inline_Narrow_Oval
- R1, R2, R3: renamed from R?; footprint (none) -> Resistors_ThroughHole:Resistor_Horizontal_RM20mm
- U1: footprint (none) -> Pin_Headers:Pin_Header_Angled_2x03
Changed lines of the file:
@@
 F 0 "IC1" H 1750 3600 50  0000 L BNN
 F 1 "ATMEGA328-P" H 2900 950 50  0000 L BNN
-F 2 "DIL28" H 2500 2350 50  0000 C CIN
+F 2 "Housings_DIP:DIP-28_W7.62mm" H 2500 2350 50  0000 C CIN
 F 3 "" H 2500 2350 50  0000 C CNN
 	1    2500 2350
@@
 F 0 "U1" H 8600 3400 60  0000 C CNN
 F 1 "BlueSmirf" H 8750 3750 60  0000 C TNN
-F 2 "" H 8800 3550 60  0000 C CNN
+F 2 "Pin_Headers:Pin_Header_Angled_2x03" H 8800 3550 60  0001 C CNN
 F 3 "" H 8800 3550 60  0000 C CNN
 	1    8800 3550
@@
 $EndComp
 $Comp
-L GND #PWR1
+L GND #PWR01
 U 1 1 5715DC43
 P 1500 3800
-F 0 "#PWR1" H 1500 3550 50  0001 C CNN
+F 0 "#PWR01" H 1500 3550 50  0001 C CNN
 F 1 "GND" H 1500 3650 50  0000 C CNN
 F 2 "" H 1500 3800 50  0000 C CNN
@@
 $EndSheet
 $Comp
-L Q_NPN_BCE Q?
+L Q_NPN_BCE Q1
 U 1 1 571628D5
 P 10000 1750
-F 0 "Q?" H 10300 1800 50  0000 R CNN
+F 0 "Q1" H 10300 1800 50  0000 R CNN
 F 1 "Q_NPN_BCE" H 10600 1700 50  0000 R CNN
-F 2 "" H 10200 1850 50  0000 C CNN
+F 2 "TO_SOT_Packages_THT:TO-92_Inline_Narrow_Oval" H 10200 1850 50  0001 C CNN
 F 3 "" H 10000 1750 50  0000 C CNN
 	1    10000 1750
@@
 	10100 1950 10100 2450
 $Comp
-L GND #PWR?
+L GND #PWR02
 U 1 1 571629AA
 P 10100 2450
-F 0 "#PWR?" H 10100 2200 50  0001 C CNN
+F 0 "#PWR02" H 10100 2200 50  0001 C CNN
 F 1 "GND" H 10100 2300 50  0000 C CNN
 F 2 "" H 10100 2450 50  0000 C CNN
@@
 $EndComp
 $Comp
-L R R?
+L R R3
 U 1 1 571629D2
 P 10100 1150
-F 0 "R?" V 10180 1150 50  0000 C CNN
+F 0 "R3" V 10180 1150 50  0000 C CNN
 F 1 "R" V 10100 1150 50  0000 C CNN
-F 2 "" V 10030 1150 50  0000 C CNN
+F 2 "Resistors_ThroughHole:Resistor_Horizontal_RM20mm" V 10030 1150 50  0001 C CNN
 F 3 "" H 10100 1150 50  0000 C CNN
 	1    10100 1150
@@
 $EndSheet
 Wire Wire Line
-	8200 5400 8200 5000
-Wire Wire Line
-	8200 5000 7450 5000
+	8200 5000 8200 5400
+Wire Wire Line
+	7450 5000 8200 5000
 Wire Wire Line
 	8000 5000 8000 5850
@@
 	8850 4900 8800 4900
 $Comp
-L GND #PWR?
+L GND #PWR03
 U 1 1 57165880
 P 8800 4900
-F 0 "#PWR?" H 8800 4650 50  0001 C CNN
+F 0 "#PWR03" H 8800 4650 50  0001 C CNN
 F 1 "GND" H 8800 4750 50  0000 C CNN
 F 2 "" H 8800 4900 50  0000 C CNN
@@
 	5200 1150 5750 1150
 $Comp
-L Photores R?
+L Photores R2
 U 1 1 5716DAD8
 P 5000 2300
-F 0 "R?" V 5080 2300 50  0000 C CNN
+F 0 "R2" V 5080 2300 50  0000 C CNN
 F 1 "Photores" V 5210 2300 50  0000 C TNN
-F 2 "" V 4930 2300 50  0000 C CNN
+F 2 "Resistors_ThroughHole:Resistor_Horizontal_RM20mm" V 4930 2300 50  0001 C CNN
 F 3 "" H 5000 2300 50  0000 C CNN
 	1    5000 2300
@@
 $EndComp
 $Comp
-L R R?
+L R R1
 U 1 1 5716E4CF
 P 4450 2050
-F 0 "R?" V 4530 2050 50  0000 C CNN
+F 0 "R1" V 4530 2050 50  0000 C CNN
 F 1 "10k" V 4450 2050 50  0000 C CNN
-F 2 "" V 4380 2050 50  0000 C CNN
+F 2 "Resistors_ThroughHole:Resistor_Horizontal_RM20mm" V 4380 2050 50  0001 C CNN
 F 3 "" H 4450 2050 50  0000 C CNN
 	1    4450 2050
@@
 Connection ~ 5500 1150
 Wire Wire Line
-	4750 2300 4150 2300
+	4150 2300 4750 2300
 Wire Wire Line
 	4150 2300 4150 2100
@@
 	4150 2100 3500 2100
 $Comp
-L GND #PWR?
+L GND #PWR04
 U 1 1 5716EE89
 P 4450 1800
-F 0 "#PWR?" H 4450 1550 50  0001 C CNN
+F 0 "#PWR04" H 4450 1550 50  0001 C CNN
 F 1 "GND" H 4450 1650 50  0000 C CNN
 F 2 "" H 4450 1800 50  0000 C CNN
@@
 	8350 4800 7450 4800
 Wire Wire Line
-	9500 5200 7700 5200
+	7700 5200 9500 5200
 Wire Wire Line
 	7700 5200 7700 5500
