File: KiCad/Project.sch (KiCad schematic (older format))
At the start: 11 parts, among them IC1 ATMEGA328-P, P1 CONN_02X03, P2 CONN_01X02, SW4 SW_PUSH, U1 BlueSmirf, Y1 Crystal

Commit message: Revert "Added smaller footprints"
This reverts commit 0613a684753a289cb87120d105616d3a60c555f9.
Parts:
- R3, SW4: footprint Wire_Pads:SolderWirePad_2x_1mmDrill -> Wire_Connections_Bridges:WireConnection_1.50mmDrill
Changed lines of the file:
@@
 $EndComp
 $Comp
-L GND #PWR01
+L GND #PWR1
 U 1 1 5715DC43
 P 1500 3800
-F 0 "#PWR01" H 1500 3550 50  0001 C CNN
+F 0 "#PWR1" H 1500 3550 50  0001 C CNN
 F 1 "GND" H 1500 3650 50  0000 C CNN
 F 2 "" H 1500 3800 50  0000 C CNN
@@
 	8850 4900 8800 4900
 $Comp
-L GND #PWR02
+L GND #PWR7
 U 1 1 57165880
 P 8800 4900
-F 0 "#PWR02" H 8800 4650 50  0001 C CNN
+F 0 "#PWR7" H 8800 4650 50  0001 C CNN
 F 1 "GND" H 8800 4750 50  0000 C CNN
 F 2 "" H 8800 4900 50  0000 C CNN
@@
 F 0 "R3" V 5080 2300 50  0000 C CNN
 F 1 "Photores" V 5210 2300 50  0000 C TNN
-F 2 "Wire_Pads:SolderWirePad_2x_1mmDrill" V 4930 2300 50  0001 C CNN
+F 2 "Wire_Connections_Bridges:WireConnection_1.50mmDrill" V 4930 2300 50  0001 C CNN
 F 3 "" H 5000 2300 50  0000 C CNN
 	1    5000 2300
@@
 	4150 2100 3500 2100
 $Comp
-L GND #PWR03
+L GND #PWR4
 U 1 1 5716EE89
 P 4450 1800
-F 0 "#PWR03" H 4450 1550 50  0001 C CNN
+F 0 "#PWR4" H 4450 1550 50  0001 C CNN
 F 1 "GND" H 4450 1650 50  0000 C CNN
 F 2 "" H 4450 1800 50  0000 C CNN
@@
 	4300 2700 3500 2700
 $Comp
-L GND #PWR04
+L GND #PWR3
 U 1 1 5733AA01
 P 4250 1650
-F 0 "#PWR04" H 4250 1400 50  0001 C CNN
+F 0 "#PWR3" H 4250 1400 50  0001 C CNN
 F 1 "GND" H 4250 1500 50  0000 C CNN
 F 2 "" H 4250 1650 50  0000 C CNN
@@
 $EndComp
 $Comp
-L GND #PWR05
+L GND #PWR5
 U 1 1 5733D1EA
 P 6650 2300
-F 0 "#PWR05" H 6650 2050 50  0001 C CNN
+F 0 "#PWR5" H 6650 2050 50  0001 C CNN
 F 1 "GND" H 6650 2150 50  0000 C CNN
 F 2 "" H 6650 2300 50  0000 C CNN
@@
 $EndComp
 $Comp
-L GND #PWR06
+L GND #PWR6
 U 1 1 5733D278
 P 6850 2650
-F 0 "#PWR06" H 6850 2400 50  0001 C CNN
+F 0 "#PWR6" H 6850 2400 50  0001 C CNN
 F 1 "GND" H 6850 2500 50  0000 C CNN
 F 2 "" H 6850 2650 50  0000 C CNN
@@
 F 0 "SW4" H 4150 4310 50  0000 C CNN
 F 1 "SW_PUSH" H 4000 4120 50  0000 C CNN
-F 2 "Wire_Pads:SolderWirePad_2x_1mmDrill" H 4000 4200 50  0001 C CNN
+F 2 "Wire_Connections_Bridges:WireConnection_1.50mmDrill" H 4000 4200 50  0001 C CNN
 F 3 "" H 4000 4200 50  0000 C CNN
 	1    4000 4200
@@
 $EndComp
 $Comp
-L GND #PWR07
+L GND #PWR2
 U 1 1 5734269F
 P 3650 4700
-F 0 "#PWR07" H 3650 4450 50  0001 C CNN
+F 0 "#PWR2" H 3650 4450 50  0001 C CNN
 F 1 "GND" H 3650 4550 50  0000 C CNN
 F 2 "" H 3650 4700 50  0000 C CNN
