File: KiCad/VoltRegulator.sch (KiCad schematic (older format))
At the start: 10 parts

Commit message: Added tasklist explenation
Parts:
- C1, C3: renamed from C?; footprint (none) -> Capacitors_ThroughHole:C_Disc_D6_P5
- C2, C4: renamed from C?; footprint (none) -> Capacitors_ThroughHole:C_Radial_D5_L11_P2.5
- R4, R5, R6, R7: renamed from R?; footprint (none) -> Resistors_ThroughHole:Resistor_Horizontal_RM20mm
- U2, U3: renamed from U?; footprint (none) -> TO_SOT_Packages_THT:TO-220_Neutral123_Vertical
Changed lines of the file:
@@
 $EndDescr
 $Comp
-L LM317_SOT223 U?
+L LM317_SOT223 U2
 U 1 1 57160D0E
 P 4050 2600
-F 0 "U?" H 4050 2900 50  0000 C CNN
+F 0 "U2" H 4050 2900 50  0000 C CNN
 F 1 "LM317" H 4100 2350 50  0000 L CNN
-F 2 "" H 4050 2600 50  0000 C CNN
+F 2 "TO_SOT_Packages_THT:TO-220_Neutral123_Vertical" H 4050 2600 50  0001 C CNN
 F 3 "" H 4050 2600 50  0000 C CNN
 	1    4050 2600
@@
 $EndComp
 $Comp
-L +9V #PWR?
+L +9V #PWR05
 U 1 1 571610CA
 P 2800 2000
-F 0 "#PWR?" H 2800 1850 50  0001 C CNN
+F 0 "#PWR05" H 2800 1850 50  0001 C CNN
 F 1 "+9V" H 2800 2140 50  0000 C CNN
 F 2 "" H 2800 2000 50  0000 C CNN
@@
 $EndComp
 $Comp
-L R R?
+L R R5
 U 1 1 57161132
 P 4650 2750
-F 0 "R?" V 4730 2750 50  0000 C CNN
+F 0 "R5" V 4730 2750 50  0000 C CNN
 F 1 "330" V 4650 2750 50  0000 C CNN
-F 2 "" V 4580 2750 50  0000 C CNN
+F 2 "Resistors_ThroughHole:Resistor_Horizontal_RM20mm" V 4580 2750 50  0001 C CNN
 F 3 "" H 4650 2750 50  0000 C CNN
 	1    4650 2750
@@
 $EndComp
 $Comp
-L R R?
+L R R4
 U 1 1 5716119D
 P 4050 3300
-F 0 "R?" V 4130 3300 50  0000 C CNN
+F 0 "R4" V 4130 3300 50  0000 C CNN
 F 1 "1K" V 4050 3300 50  0000 C CNN
-F 2 "" V 3980 3300 50  0000 C CNN
+F 2 "Resistors_ThroughHole:Resistor_Horizontal_RM20mm" V 3980 3300 50  0001 C CNN
 F 3 "" H 4050 3300 50  0000 C CNN
 	1    4050 3300
@@
 5V
 $Comp
-L GND #PWR?
+L GND #PWR06
 U 1 1 571613A6
 P 4050 3550
-F 0 "#PWR?" H 4050 3300 50  0001 C CNN
+F 0 "#PWR06" H 4050 3300 50  0001 C CNN
 F 1 "GND" H 4050 3400 50  0000 C CNN
 F 2 "" H 4050 3550 50  0000 C CNN
@@
 $EndComp
 $Comp
-L LM317_SOT223 U?
+L LM317_SOT223 U3
 U 1 1 571810AE
 P 7750 2600
-F 0 "U?" H 7750 2900 50  0000 C CNN
+F 0 "U3" H 7750 2900 50  0000 C CNN
 F 1 "LM317" H 7800 2350 50  0000 L CNN
-F 2 "" H 7750 2600 50  0000 C CNN
+F 2 "TO_SOT_Packages_THT:TO-220_Neutral123_Vertical" H 7750 2600 50  0001 C CNN
 F 3 "" H 7750 2600 50  0000 C CNN
 	1    7750 2600
@@
 $EndComp
 $Comp
-L +9V #PWR?
+L +9V #PWR07
 U 1 1 571810B4
 P 6500 2000
-F 0 "#PWR?" H 6500 1850 50  0001 C CNN
+F 0 "#PWR07" H 6500 1850 50  0001 C CNN
 F 1 "+9V" H 6500 2140 50  0000 C CNN
 F 2 "" H 6500 2000 50  0000 C CNN
@@
 $EndComp
 $Comp
-L R R?
+L R R7
 U 1 1 571810BA
 P 8350 2800
-F 0 "R?" V 8430 2800 50  0000 C CNN
+F 0 "R7" V 8430 2800 50  0000 C CNN
 F 1 "330" V 8350 2800 50  0000 C CNN
-F 2 "" V 8280 2800 50  0000 C CNN
+F 2 "Resistors_ThroughHole:Resistor_Horizontal_RM20mm" V 8280 2800 50  0001 C CNN
 F 3 "" H 8350 2800 50  0000 C CNN
 	1    8350 2800
@@
 $EndComp
 $Comp
-L R R?
+L R R6
 U 1 1 571810C0
 P 7750 3300
-F 0 "R?" V 7830 3300 50  0000 C CNN
+F 0 "R6" V 7830 3300 50  0000 C CNN
 F 1 "470" V 7750 3300 50  0000 C CNN
-F 2 "" V 7680 3300 50  0000 C CNN
+F 2 "Resistors_ThroughHole:Resistor_Horizontal_RM20mm" V 7680 3300 50  0001 C CNN
 F 3 "" H 7750 3300 50  0000 C CNN
 	1    7750 3300
@@
 3V
 $Comp
-L GND #PWR?
+L GND #PWR08
 U 1 1 571810D3
 P 7750 3550
-F 0 "#PWR?" H 7750 3300 50  0001 C CNN
+F 0 "#PWR08" H 7750 3300 50  0001 C CNN
 F 1 "GND" H 7750 3400 50  0000 C CNN
 F 2 "" H 7750 3550 50  0000 C CNN
@@
 	4050 3450 4050 3550
 $Comp
-L CP1 C?
+L CP1 C2
 U 1 1 571BB487
 P 5100 2750
-F 0 "C?" H 5125 2850 50  0000 L CNN
+F 0 "C2" H 5125 2850 50  0000 L CNN
 F 1 "1uF" H 5125 2650 50  0000 L CNN
-F 2 "" H 5100 2750 50  0000 C CNN
+F 2 "Capacitors_ThroughHole:C_Radial_D5_L11_P2.5" H 5100 2750 50  0001 C CNN
 F 3 "" H 5100 2750 50  0000 C CNN
 	1    5100 2750
@@
 $EndComp
 $Comp
-L CP1 C?
+L CP1 C4
 U 1 1 571BB503
 P 8850 2800
-F 0 "C?" H 8875 2900 50  0000 L CNN
+F 0 "C4" H 8875 2900 50  0000 L CNN
 F 1 "1uF" H 8875 2700 50  0000 L CNN
-F 2 "" H 8850 2800 50  0000 C CNN
+F 2 "Capacitors_ThroughHole:C_Radial_D5_L11_P2.5" H 8850 2800 50  0001 C CNN
 F 3 "" H 8850 2800 50  0000 C CNN
 	1    8850 2800
@@
 	8850 2950 8850 3050
 $Comp
-L C C?
+L C C1
 U 1 1 571BBB0A
 P 3350 2750
-F 0 "C?" H 3375 2850 50  0000 L CNN
+F 0 "C1" H 3375 2850 50  0000 L CNN
 F 1 "0.1uF" H 3375 2650 50  0000 L CNN
-F 2 "" H 3388 2600 50  0000 C CNN
+F 2 "Capacitors_ThroughHole:C_Disc_D6_P5" H 3388 2600 50  0001 C CNN
 F 3 "" H 3350 2750 50  0000 C CNN
 	1    3350 2750
@@
 $EndComp
 $Comp
-L C C?
+L C C3
 U 1 1 571BBC58
 P 7050 2800
-F 0 "C?" H 7075 2900 50  0000 L CNN
+F 0 "C3" H 7075 2900 50  0000 L CNN
 F 1 "0.1uF" H 7075 2700 50  0000 L CNN
-F 2 "" H 7088 2650 50  0000 C CNN
+F 2 "Capacitors_ThroughHole:C_Disc_D6_P5" H 7088 2650 50  0001 C CNN
 F 3 "" H 7050 2800 50  0000 C CNN
 	1    7050 2800
@@
 	3350 2900 3350 3050
 $Comp
-L GND #PWR?
+L GND #PWR09
 U 1 1 571BC1AC
 P 3350 3050
-F 0 "#PWR?" H 3350 2800 50  0001 C CNN
+F 0 "#PWR09" H 3350 2800 50  0001 C CNN
 F 1 "GND" H 3350 2900 50  0000 C CNN
 F 2 "" H 3350 3050 50  0000 C CNN
@@
 $EndComp
 $Comp
-L GND #PWR?
+L GND #PWR010
 U 1 1 571BC2DA
 P 5100 3050
-F 0 "#PWR?" H 5100 2800 50  0001 C CNN
+F 0 "#PWR010" H 5100 2800 50  0001 C CNN
 F 1 "GND" H 5100 2900 50  0000 C CNN
 F 2 "" H 5100 3050 50  0000 C CNN
@@
 $EndComp
 $Comp
-L GND #PWR?
+L GND #PWR011
 U 1 1 571BC41B
 P 7050 3050
-F 0 "#PWR?" H 7050 2800 50  0001 C CNN
+F 0 "#PWR011" H 7050 2800 50  0001 C CNN
 F 1 "GND" H 7050 2900 50  0000 C CNN
 F 2 "" H 7050 3050 50  0000 C CNN
@@
 $EndComp
 $Comp
-L GND #PWR?
+L GND #PWR012
 U 1 1 571BC444
 P 8850 3050
-F 0 "#PWR?" H 8850 2800 50  0001 C CNN
+F 0 "#PWR012" H 8850 2800 50  0001 C CNN
 F 1 "GND" H 8850 2900 50  0000 C CNN
 F 2 "" H 8850 3050 50  0000 C CNN
