File: KiCad/IR.sch (KiCad schematic (older format))
At the start: 34 parts, among them IC2 ATTINY85-P, IC3 ATTINY85-P, P3 CONN_01X02, P4 CONN_01X02, P5 CONN_02X04, P6 CONN_02X03, Q1 Q_NPN_BCE, Q2 Q_NPN_BCE

Commit message: Updated the pcb to smaller size and footprints
Parts:
- D1, D10, D11, D12, D2, D3, D4, D5, D6, D7, D8, D9: footprint Wire_Pads:SolderWirePad_2x_1mmDrill -> Holes:SolderWirePad1mmmodified
Changed lines of the file:
@@
 SCL
 $Comp
-L GND #PWR015
+L GND #PWR017
 U 1 1 57175BA8
 P 8650 1700
-F 0 "#PWR015" H 8650 1450 50  0001 C CNN
+F 0 "#PWR017" H 8650 1450 50  0001 C CNN
 F 1 "GND" H 8650 1550 50  0000 C CNN
 F 2 "" H 8650 1700 50  0000 C CNN
@@
 F 0 "D9" H 3300 2900 50  0000 C CNN
 F 1 "IR_Recieve" H 3316 2633 50  0000 C CNN
-F 2 "Wire_Pads:SolderWirePad_2x_1mmDrill" H 3300 2800 50  0001 C CNN
+F 2 "Holes:SolderWirePad1mmmodified" H 3300 2800 50  0001 C CNN
 F 3 "" H 3300 2800 50  0000 C CNN
 	1    3300 2800
@@
 F 0 "D7" H 2900 2900 50  0000 C CNN
 F 1 "LED" V 2900 2700 50  0000 C CNN
-F 2 "Wire_Pads:SolderWirePad_2x_1mmDrill" H 2900 2800 50  0001 C CNN
+F 2 "Holes:SolderWirePad1mmmodified" H 2900 2800 50  0001 C CNN
 F 3 "" H 2900 2800 50  0000 C CNN
 	1    2900 2800
@@
 F 0 "D11" H 3700 2900 50  0000 C CNN
 F 1 "LED" V 3700 2700 50  0000 C CNN
-F 2 "Wire_Pads:SolderWirePad_2x_1mmDrill" H 3700 2800 50  0001 C CNN
+F 2 "Holes:SolderWirePad1mmmodified" H 3700 2800 50  0001 C CNN
 F 3 "" H 3700 2800 50  0000 C CNN
 	1    3700 2800
@@
 F 0 "D3" H 1800 2900 50  0000 C CNN
 F 1 "IR_Recieve" H 1816 2633 50  0000 C CNN
-F 2 "Wire_Pads:SolderWirePad_2x_1mmDrill" H 1800 2800 50  0001 C CNN
+F 2 "Holes:SolderWirePad1mmmodified" H 1800 2800 50  0001 C CNN
 F 3 "" H 1800 2800 50  0000 C CNN
 	1    1800 2800
@@
 F 0 "D1" H 1400 2900 50  0000 C CNN
 F 1 "LED" V 1400 2700 50  0000 C CNN
-F 2 "Wire_Pads:SolderWirePad_2x_1mmDrill" H 1400 2800 50  0001 C CNN
+F 2 "Holes:SolderWirePad1mmmodified" H 1400 2800 50  0001 C CNN
 F 3 "" H 1400 2800 50  0000 C CNN
 	1    1400 2800
@@
 F 0 "D5" H 2200 2900 50  0000 C CNN
 F 1 "LED" V 2200 2700 50  0000 C CNN
-F 2 "Wire_Pads:SolderWirePad_2x_1mmDrill" H 2200 2800 50  0001 C CNN
+F 2 "Holes:SolderWirePad1mmmodified" H 2200 2800 50  0001 C CNN
 F 3 "" H 2200 2800 50  0000 C CNN
 	1    2200 2800
@@
 $EndComp
 $Comp
-L GND #PWR016
+L GND #PWR018
 U 1 1 57175C1F
 P 4000 3400
-F 0 "#PWR016" H 4000 3150 50  0001 C CNN
+F 0 "#PWR018" H 4000 3150 50  0001 C CNN
 F 1 "GND" H 4000 3250 50  0000 C CNN
 F 2 "" H 4000 3400 50  0000 C CNN
@@
 Text HLabel 5600 1050 0    60   BiDi ~ 0
 SDA
-Text HLabel 9050 1050 2    60   Input ~ 0
+Text HLabel 8550 1050 2    60   Input ~ 0
 5V
 Text HLabel 1400 2100 1    60   Input ~ 0
@@
 Text HLabel 3700 2100 1    60   Input ~ 0
 3V
-Wire Wire Line
-	9050 1050 8550 1050
-Wire Wire Line
-	8550 1550 8650 1550
-Wire Wire Line
-	8650 1550 8650 1700
 Wire Wire Line
 	3300 1900 3300 2100
@@
 SCL
 $Comp
-L GND #PWR017
+L GND #PWR019
 U 1 1 5735BAD5
 P 8700 5100
-F 0 "#PWR017" H 8700 4850 50  0001 C CNN
+F 0 "#PWR019" H 8700 4850 50  0001 C CNN
 F 1 "GND" H 8700 4950 50  0000 C CNN
 F 2 "" H 8700 5100 50  0000 C CNN
@@
 F 0 "D10" H 3350 6300 50  0000 C CNN
 F 1 "IR_Recieve" H 3366 6033 50  0000 C CNN
-F 2 "Wire_Pads:SolderWirePad_2x_1mmDrill" H 3350 6200 50  0001 C CNN
+F 2 "Holes:SolderWirePad1mmmodified" H 3350 6200 50  0001 C CNN
 F 3 "" H 3350 6200 50  0000 C CNN
 	1    3350 6200
@@
 F 0 "D8" H 2950 6300 50  0000 C CNN
 F 1 "LED" V 2950 6100 50  0000 C CNN
-F 2 "Wire_Pads:SolderWirePad_2x_1mmDrill" H 2950 6200 50  0001 C CNN
+F 2 "Holes:SolderWirePad1mmmodified" H 2950 6200 50  0001 C CNN
 F 3 "" H 2950 6200 50  0000 C CNN
 	1    2950 6200
@@
 F 0 "D12" H 3750 6300 50  0000 C CNN
 F 1 "LED" V 3750 6100 50  0000 C CNN
-F 2 "Wire_Pads:SolderWirePad_2x_1mmDrill" H 3750 6200 50  0001 C CNN
+F 2 "Holes:SolderWirePad1mmmodified" H 3750 6200 50  0001 C CNN
 F 3 "" H 3750 6200 50  0000 C CNN
 	1    3750 6200
@@
 F 0 "D4" H 1850 6300 50  0000 C CNN
 F 1 "IR_Recieve" H 1866 6033 50  0000 C CNN
-F 2 "Wire_Pads:SolderWirePad_2x_1mmDrill" H 1850 6200 50  0001 C CNN
+F 2 "Holes:SolderWirePad1mmmodified" H 1850 6200 50  0001 C CNN
 F 3 "" H 1850 6200 50  0000 C CNN
 	1    1850 6200
@@
 F 0 "D2" H 1450 6300 50  0000 C CNN
 F 1 "LED" V 1450 6100 50  0000 C CNN
-F 2 "Wire_Pads:SolderWirePad_2x_1mmDrill" H 1450 6200 50  0001 C CNN
+F 2 "Holes:SolderWirePad1mmmodified" H 1450 6200 50  0001 C CNN
 F 3 "" H 1450 6200 50  0000 C CNN
 	1    1450 6200
@@
 F 0 "D6" H 2250 6300 50  0000 C CNN
 F 1 "LED" V 2250 6100 50  0000 C CNN
-F 2 "Wire_Pads:SolderWirePad_2x_1mmDrill" H 2250 6200 50  0001 C CNN
+F 2 "Holes:SolderWirePad1mmmodified" H 2250 6200 50  0001 C CNN
 F 3 "" H 2250 6200 50  0000 C CNN
 	1    2250 6200
@@
 $EndComp
 $Comp
-L GND #PWR018
+L GND #PWR020
 U 1 1 5735BB1E
 P 4050 6800
-F 0 "#PWR018" H 4050 6550 50  0001 C CNN
+F 0 "#PWR020" H 4050 6550 50  0001 C CNN
 F 1 "GND" H 4050 6650 50  0000 C CNN
 F 2 "" H 4050 6800 50  0000 C CNN
@@
 Text HLabel 5600 4450 0    60   BiDi ~ 0
 SDA
-Text HLabel 9100 4450 2    60   Input ~ 0
+Text HLabel 8600 4450 2    60   Input ~ 0
 5V
 Text HLabel 1450 5500 1    60   Input ~ 0
@@
 Text HLabel 3750 5500 1    60   Input ~ 0
 3V
-Wire Wire Line
-	9100 4450 8600 4450
 Wire Wire Line
 	8600 4950 8700 4950
@@
 Connection ~ 9300 3850
 $Comp
-L GND #PWR019
+L GND #PWR021
 U 1 1 5735C5A5
 P 9300 2950
-F 0 "#PWR019" H 9300 2700 50  0001 C CNN
+F 0 "#PWR021" H 9300 2700 50  0001 C CNN
 F 1 "GND" H 9300 2800 50  0000 C CNN
 F 2 "" H 9300 2950 50  0000 C CNN
@@
 Wire Wire Line
 	5700 4550 5900 4550
+Wire Wire Line
+	8650 1700 8650 1550
+Wire Wire Line
+	8650 1550 8550 1550
 $EndSCHEMATC
