File: KiCad/Lights.sch (KiCad schematic (older format))
At the start: 12 parts, among them Q4 Q_NPN_BCE, Q5 NPN

Commit message: Added smaller footprints
Parts:
- D13, D14, D15, D16: footprint Wire_Connections_Bridges:WireConnection_1.50mmDrill -> Wire_Pads:SolderWirePad_2x_1mmDrill
Changed lines of the file:
@@
 F 0 "D13" H 5100 1450 50  0000 C CNN
 F 1 "LED" H 5100 1250 50  0000 C CNN
-F 2 "Wire_Connections_Bridges:WireConnection_1.50mmDrill" H 5100 1350 50  0001 C CNN
+F 2 "Wire_Pads:SolderWirePad_2x_1mmDrill" H 5100 1350 50  0001 C CNN
 F 3 "" H 5100 1350 50  0000 C CNN
 	1    5100 1350
@@
 F 0 "D15" H 5650 1450 50  0000 C CNN
 F 1 "LED" H 5650 1250 50  0000 C CNN
-F 2 "Wire_Connections_Bridges:WireConnection_1.50mmDrill" H 5650 1350 50  0001 C CNN
+F 2 "Wire_Pads:SolderWirePad_2x_1mmDrill" H 5650 1350 50  0001 C CNN
 F 3 "" H 5650 1350 50  0000 C CNN
 	1    5650 1350
@@
 F 0 "D14" H 5350 4200 50  0000 C CNN
 F 1 "LED" H 5350 4000 50  0000 C CNN
-F 2 "Wire_Connections_Bridges:WireConnection_1.50mmDrill" H 5350 4100 50  0001 C CNN
+F 2 "Wire_Pads:SolderWirePad_2x_1mmDrill" H 5350 4100 50  0001 C CNN
 F 3 "" H 5350 4100 50  0000 C CNN
 	1    5350 4100
@@
 F 0 "D16" H 5900 4200 50  0000 C CNN
 F 1 "LED" H 5900 4000 50  0000 C CNN
-F 2 "Wire_Connections_Bridges:WireConnection_1.50mmDrill" H 5900 4100 50  0001 C CNN
+F 2 "Wire_Pads:SolderWirePad_2x_1mmDrill" H 5900 4100 50  0001 C CNN
 F 3 "" H 5900 4100 50  0000 C CNN
 	1    5900 4100
@@
 $EndComp
 $Comp
-L GND #PWR21
+L GND #PWR020
 U 1 1 57167CC8
 P 4600 2600
-F 0 "#PWR21" H 4600 2350 50  0001 C CNN
+F 0 "#PWR020" H 4600 2350 50  0001 C CNN
 F 1 "GND" H 4600 2450 50  0000 C CNN
 F 2 "" H 4600 2600 50  0000 C CNN
@@
 $EndComp
 $Comp
-L GND #PWR20
+L GND #PWR021
 U 1 1 57168248
 P 4200 3300
-F 0 "#PWR20" H 4200 3050 50  0001 C CNN
+F 0 "#PWR021" H 4200 3050 50  0001 C CNN
 F 1 "GND" H 4200 3150 50  0000 C CNN
 F 2 "" H 4200 3300 50  0000 C CNN

Commit message: Updated the pcb to smaller size and footprints
Parts:
- D13, D14, D15, D16: footprint Wire_Pads:SolderWirePad_2x_1mmDrill -> Holes:SolderWirePad1mmmodified
Changed lines of the file:
@@
 F 0 "D13" H 5100 1450 50  0000 C CNN
 F 1 "LED" H 5100 1250 50  0000 C CNN
-F 2 "Wire_Pads:SolderWirePad_2x_1mmDrill" H 5100 1350 50  0001 C CNN
+F 2 "Holes:SolderWirePad1mmmodified" H 5100 1350 50  0001 C CNN
 F 3 "" H 5100 1350 50  0000 C CNN
 	1    5100 1350
@@
 F 0 "D15" H 5650 1450 50  0000 C CNN
 F 1 "LED" H 5650 1250 50  0000 C CNN
-F 2 "Wire_Pads:SolderWirePad_2x_1mmDrill" H 5650 1350 50  0001 C CNN
+F 2 "Holes:SolderWirePad1mmmodified" H 5650 1350 50  0001 C CNN
 F 3 "" H 5650 1350 50  0000 C CNN
 	1    5650 1350
@@
 F 0 "D14" H 5350 4200 50  0000 C CNN
 F 1 "LED" H 5350 4000 50  0000 C CNN
-F 2 "Wire_Pads:SolderWirePad_2x_1mmDrill" H 5350 4100 50  0001 C CNN
+F 2 "Holes:SolderWirePad1mmmodified" H 5350 4100 50  0001 C CNN
 F 3 "" H 5350 4100 50  0000 C CNN
 	1    5350 4100
@@
 F 0 "D16" H 5900 4200 50  0000 C CNN
 F 1 "LED" H 5900 4000 50  0000 C CNN
-F 2 "Wire_Pads:SolderWirePad_2x_1mmDrill" H 5900 4100 50  0001 C CNN
+F 2 "Holes:SolderWirePad1mmmodified" H 5900 4100 50  0001 C CNN
 F 3 "" H 5900 4100 50  0000 C CNN
 	1    5900 4100
@@
 $EndComp
 $Comp
-L GND #PWR020
+L GND #PWR022
 U 1 1 57167CC8
 P 4600 2600
-F 0 "#PWR020" H 4600 2350 50  0001 C CNN
+F 0 "#PWR022" H 4600 2350 50  0001 C CNN
 F 1 "GND" H 4600 2450 50  0000 C CNN
 F 2 "" H 4600 2600 50  0000 C CNN
@@
 $EndComp
 $Comp
-L GND #PWR021
+L GND #PWR023
 U 1 1 57168248
 P 4200 3300
-F 0 "#PWR021" H 4200 3050 50  0001 C CNN
+F 0 "#PWR023" H 4200 3050 50  0001 C CNN
 F 1 "GND" H 4200 3150 50  0000 C CNN
 F 2 "" H 4200 3300 50  0000 C CNN
